File: QuadcopterHardware/Quadcopter/Quadcopter.sch (EAGLE design)
At the start: 13 parts, among them M1 WIRELESS-NRF24L01, U1 ATMEGA328P_TQFP, U2 TC1262-3.3VDB

Commit message: added to schematic...almost done :)
Parts:
- removed MR.DIODE: DB2W40300L, quad:DB2W40300L
- removed MS.MOSFET: N-CHANNEL-MOSFET-IRLML6244TRPBF, quad:N-CHANNEL-MOSFET-IRLML6244TRPBF
- added C3, C4, C5, C6: 100nF, rcl:C-USC0603
- added FLYBACK_DIODE1, FLYBACK_DIODE2, FLYBACK_DIODE3, FLYBACK_DIODE4: DB2W40300L, quad:DB2W40300L
- added J2: FTDI_DEVICERA_SMT, quad:FTDI_DEVICERA_SMT
- added MOSFET1, MOSFET2, MOSFET3, MOSFET4: N-CHANNEL-MOSFET-IRLML6244TRPBF, quad:N-CHANNEL-MOSFET-IRLML6244TRPBF
- added MOTOR1, MOTOR2, MOTOR3: JST_CONNECTOR_FEMALE, quad:JST_CONNECTOR_FEMALE
- added R3, R4, R5: 10K Ohms, rcl:R-US_0204/5
- added U3: GY-521MPU6050, quad:GY-521MPU6050
Connections:
- removed net DRAIN: MOTOR.-, MR.DIODE.PPIN, MS.MOSFET.D
- removed net N$1: R2.1, S1.2, U1.PC6(/RESET)
- removed net N$3: U1.PD6(AIN0)
- new net DRAIN1: FLYBACK_DIODE1.PPIN, MOSFET1.D, MOTOR.-
- new net DRAIN2: FLYBACK_DIODE2.PPIN, MOSFET2.D, MOTOR1.-
- new net DRAIN3: FLYBACK_DIODE3.PPIN, MOSFET3.D, MOTOR2.-
- new net DRAIN4: FLYBACK_DIODE4.PPIN, MOSFET4.D, MOTOR3.-
- new net DTR: C6.2, J2.DTR
- new net PWM2: MOSFET2.G, R3.2
- new net PWM3: MOSFET3.G, R4.2
- new net PWM4: MOSFET4.G, R5.2
- new net RST: C6.1, R2.1, S1.2, U1.PC6(/RESET)
- new net SCL: U1.PC5(ADC5/SCL), U3.SCL
- new net SDA: U1.PC4(ADC4/SDA), U3.SDA
- new net UART_RX: J2.RXI, U1.PD0(RXD)
- new net UART_TX: J2.TXO, U1.PD1(TXD)
- new net XTAL1: RES1.P$3, U1.PB6(XTAL1/TOSC1)
- new net XTAL2: RES1.P$1, U1.PB7(XTAL2/TOSC2)
- net GND: now also C3.2, C4.2, C5.2, J2.CTS, J2.GND, MOSFET1.S, MOSFET2.S, MOSFET3.S, MOSFET4.S, R3.1, R4.1, R5.1, RES1.P$2, U1.AGND, U3.GND; no longer MS.MOSFET.S
- net PWM1: now also MOSFET1.G; no longer MS.MOSFET.G
- net REGPOW: now also C3.1, C4.1, C5.1, J2.VCC, M1.VCC, U3.VCC
- net UNREGPOW: now also FLYBACK_DIODE1.GPIN, FLYBACK_DIODE2.GPIN, FLYBACK_DIODE3.GPIN, FLYBACK_DIODE4.GPIN, MOTOR1.+, MOTOR2.+, MOTOR3.+; no longer M1.VCC, MR.DIODE.GPIN
Other:
- moved on the sheet: C1, C2, J1, M1, R1, RES1, U2

Commit message: Version 2.0 of Schematic
Parts:
- added C7: 100nF, rcl:C-USC0603
- added R6: 1.7K Ohms, rcl:R-US_0204/5
- added R7: 1K Ohms, rcl:R-US_0204/5
- C1, C2: value (none) -> 1uF
Connections:
- new net CE: M1.CE, U1.PD2(INT0)
- new net CSN: M1.CSN, U1.PD4(XCK/T0)
- new net N$1: C7.1, U1.AREF
- new net VDIV: R6.2, R7.2, U1.PC0(ADC0)
- net GND: now also C7.2, R7.1
- net PWM1: now also U1.PD3(INT1)
- net PWM2: now also U1.PD5(T1)
- net PWM3: now also U1.PD6(AIN0)
- net PWM4: now also U1.PB1(OC1A)
- net UNREGPOW: now also R6.1
Changed lines of the file:
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@@
 <part name="M1" library="quad" deviceset="WIRELESS-NRF24L01" device=""/>
 <part name="J1" library="SparkFun-Connectors" deviceset="JST_2MM_MALE" device=""/>
-<part name="C1" library="rcl" deviceset="C-US" device="C0603"/>
-<part name="C2" library="rcl" deviceset="C-US" device="C0603"/>
+<part name="C1" library="rcl" deviceset="C-US" device="C0603" value="1uF"/>
+<part name="C2" library="rcl" deviceset="C-US" device="C0603" value="1uF"/>
 <part name="R2" library="rcl" deviceset="R-US_" device="0204/5" value="10K Ohms"/>
 <part name="MOSFET2" library="quad" deviceset="N-CHANNEL-MOSFET" device="-IRLML6244TRPBF"/>
@@
 <part name="GND15" library="supply1" deviceset="GND" device=""/>
 <part name="C6" library="rcl" deviceset="C-US" device="C0603" value="100nF"/>
+<part name="C7" library="rcl" deviceset="C-US" device="C0603" value="100nF"/>
+<part name="R6" library="rcl" deviceset="R-US_" device="0204/5" value="1.7K Ohms"/>
+<part name="R7" library="rcl" deviceset="R-US_" device="0204/5" value="1K Ohms"/>
 </parts>
 <sheets>
@@
 <instance part="GND15" gate="1" x="25.4" y="35.56"/>
 <instance part="C6" gate="G$1" x="-88.9" y="114.3" rot="R90"/>
+<instance part="C7" gate="G$1" x="-109.22" y="91.44" rot="R270"/>
+<instance part="R6" gate="G$1" x="-180.34" y="124.46" rot="R90"/>
+<instance part="R7" gate="G$1" x="-170.18" y="124.46" rot="R90"/>
 </instances>
 <busses>
@@
 <pinref part="C1" gate="G$1" pin="1"/>
 <pinref part="J1" gate="G$1" pin="+"/>
-<wire x1="-220.98" y1="124.46" x2="-220.98" y2="104.14" width="0.1524" layer="91"/>
+<wire x1="-220.98" y1="124.46" x2="-220.98" y2="116.84" width="0.1524" layer="91"/>
+<wire x1="-220.98" y1="116.84" x2="-220.98" y2="104.14" width="0.1524" layer="91"/>
 <wire x1="-220.98" y1="104.14" x2="-208.28" y2="104.14" width="0.1524" layer="91"/>
 <junction x="-220.98" y="104.14"/>
 <label x="-220.98" y="121.92" size="1.778" layer="95" xref="yes"/>
+<pinref part="R6" gate="G$1" pin="1"/>
+<wire x1="-220.98" y1="116.84" x2="-180.34" y2="116.84" width="0.1524" layer="91"/>
+<wire x1="-180.34" y1="116.84" x2="-180.34" y2="119.38" width="0.1524" layer="91"/>
+<junction x="-220.98" y="116.84"/>
 </segment>
 <segment>
@@
 <wire x1="-231.14" y1="91.44" x2="-220.98" y2="91.44" width="0.1524" layer="91"/>
 <junction x="-220.98" y="91.44"/>
+<pinref part="R7" gate="G$1" pin="1"/>
+<wire x1="-170.18" y1="119.38" x2="-165.1" y2="119.38" width="0.1524" layer="91"/>
+<wire x1="-165.1" y1="119.38" x2="-165.1" y2="142.24" width="0.1524" layer="91"/>
+<wire x1="-165.1" y1="142.24" x2="-231.14" y2="142.24" width="0.1524" layer="91"/>
+<wire x1="-231.14" y1="142.24" x2="-231.14" y2="124.46" width="0.1524" layer="91"/>
+<junction x="-231.14" y="124.46"/>
 </segment>
 <segment>
@@
 <wire x1="-127" y1="66.04" x2="-127" y2="73.66" width="0.1524" layer="91"/>
 <junction x="-127" y="73.66"/>
-<wire x1="-127" y1="73.66" x2="-127" y2="81.28" width="0.1524" layer="91"/>
+<wire x1="-127" y1="73.66" x2="-127" y2="78.74" width="0.1524" layer="91"/>
 <pinref part="C5" gate="G$1" pin="2"/>
+<wire x1="-127" y1="78.74" x2="-127" y2="81.28" width="0.1524" layer="91"/>
 <wire x1="-129.54" y1="86.36" x2="-129.54" y2="81.28" width="0.1524" layer="91"/>
 <wire x1="-129.54" y1="81.28" x2="-127" y2="81.28" width="0.1524" layer="91"/>
@@
 <junction x="-129.54" y="81.28"/>
 <junction x="-139.7" y="81.28"/>
+<pinref part="C7" gate="G$1" pin="2"/>
+<wire x1="-114.3" y1="91.44" x2="-121.92" y2="91.44" width="0.1524" layer="91"/>
+<wire x1="-121.92" y1="91.44" x2="-121.92" y2="83.82" width="0.1524" layer="91"/>
+<wire x1="-121.92" y1="83.82" x2="-124.46" y2="83.82" width="0.1524" layer="91"/>
+<wire x1="-124.46" y1="83.82" x2="-124.46" y2="78.74" width="0.1524" layer="91"/>
+<wire x1="-124.46" y1="78.74" x2="-127" y2="78.74" width="0.1524" layer="91"/>
+<junction x="-127" y="78.74"/>
 </segment>
 <segment>
@@
 <label x="-213.36" y="-15.24" size="1.778" layer="95" rot="R180" xref="yes"/>
 </segment>
+<segment>
+<pinref part="U1" gate="U$1" pin="PD3(INT1)"/>
+<wire x1="-55.88" y1="76.2" x2="-48.26" y2="76.2" width="0.1524" layer="91"/>
+<label x="-48.26" y="76.2" size="1.778" layer="95" xref="yes"/>
+</segment>
 </net>
 <net name="DRAIN3" class="0">
@@
 <label x="-139.7" y="-15.24" size="1.778" layer="95" rot="R180" xref="yes"/>
 </segment>
+<segment>
+<pinref part="U1" gate="U$1" pin="PD5(T1)"/>
+<wire x1="-55.88" y1="71.12" x2="-50.8" y2="71.12" width="0.1524" layer="91"/>
+<label x="-50.8" y="71.12" size="1.778" layer="95" xref="yes"/>
+</segment>
 </net>
 <net name="PWM3" class="0">
@@
 <label x="-68.58" y="-15.24" size="1.778" layer="95" rot="R180" xref="yes"/>
 </segment>
+<segment>
+<pinref part="U1" gate="U$1" pin="PD6(AIN0)"/>
+<wire x1="-55.88" y1="68.58" x2="-48.26" y2="68.58" width="0.1524" layer="91"/>
+<label x="-48.26" y="68.58" size="1.778" layer="95" xref="yes"/>
+</segment>
 </net>
 <net name="PWM4" class="0">
@@
 <label x="0" y="-17.78" size="1.778" layer="95" rot="R180" xref="yes"/>
 </segment>
+<segment>
+<pinref part="U1" gate="U$1" pin="PB1(OC1A)"/>
+<wire x1="-55.88" y1="58.42" x2="-48.26" y2="58.42" width="0.1524" layer="91"/>
+<label x="-48.26" y="58.42" size="1.778" layer="95" xref="yes"/>
+</segment>
 </net>
 <net name="XTAL1" class="0">
@@
 </segment>
 </net>
+<net name="CSN" class="0">
+<segment>
+<pinref part="M1" gate="G$1" pin="CSN"/>
+<wire x1="-210.82" y1="63.5" x2="-213.36" y2="63.5" width="0.1524" layer="91"/>
+<label x="-213.36" y="63.5" size="1.778" layer="95" rot="R180" xref="yes"/>
+</segment>
+<segment>
+<pinref part="U1" gate="U$1" pin="PD4(XCK/T0)"/>
+<wire x1="-55.88" y1="73.66" x2="-35.56" y2="73.66" width="0.1524" layer="91"/>
+<label x="-38.1" y="73.66" size="1.778" layer="95" xref="yes"/>
+</segment>
+</net>
+<net name="CE" class="0">
+<segment>
+<pinref part="M1" gate="G$1" pin="CE"/>
+<wire x1="-210.82" y1="66.04" x2="-215.9" y2="66.04" width="0.1524" layer="91"/>
+<label x="-213.36" y="66.04" size="1.778" layer="95" rot="R180" xref="yes"/>
+</segment>
+<segment>
+<pinref part="U1" gate="U$1" pin="PD2(INT0)"/>
+<wire x1="-55.88" y1="78.74" x2="-53.34" y2="78.74" width="0.1524" layer="91"/>
+<label x="-53.34" y="78.74" size="1.778" layer="95" xref="yes"/>
+</segment>
+</net>
+<net name="N$1" class="0">
+<segment>
+<pinref part="U1" gate="U$1" pin="AREF"/>
+<wire x1="-104.14" y1="91.44" x2="-106.68" y2="91.44" width="0.1524" layer="91"/>
+<pinref part="C7" gate="G$1" pin="1"/>
+</segment>
+</net>
+<net name="VDIV" class="0">
+<segment>
+<pinref part="R6" gate="G$1" pin="2"/>
+<pinref part="R7" gate="G$1" pin="2"/>
+<wire x1="-180.34" y1="129.54" x2="-175.26" y2="129.54" width="0.1524" layer="91"/>
+<wire x1="-175.26" y1="129.54" x2="-170.18" y2="129.54" width="0.1524" layer="91"/>
+<wire x1="-175.26" y1="129.54" x2="-175.26" y2="114.3" width="0.1524" layer="91"/>
+<junction x="-175.26" y="129.54"/>
+<wire x1="-175.26" y1="114.3" x2="-170.18" y2="114.3" width="0.1524" layer="91"/>
+<label x="-170.18" y="114.3" size="1.778" layer="95" xref="yes"/>
+</segment>
+<segment>
+<pinref part="U1" gate="U$1" pin="PC0(ADC0)"/>
+<wire x1="-55.88" y1="106.68" x2="-50.8" y2="106.68" width="0.1524" layer="91"/>
+<label x="-50.8" y="106.68" size="1.778" layer="95" xref="yes"/>
+</segment>
+</net>

Commit message: updates to schematic
Parts:
- removed R5: 10K Ohms, rcl:R-US_0204/5
- removed U2: TC1262-3.3VDB, quad:TC1262-3.3VDB
- added C9: 10uF, rcl:C-USC0603
- added LED1: RED, led:LEDCHIP-LED0603
- added LED2: GREEN, led:LEDCHIP-LED0603
- added LED3: YELLOW, led:LEDCHIP-LED0603
- added R10, R11: 10K, rcl:R-US_R0603
- added R8: 1K, rcl:R-US_R0603
- added R9: 1.7K, rcl:R-US_R0603
- added U$1: MCP1802T-3302I/OT, quad:MCP1802T-3002I/OT
- R1, R3, R4: value 10K Ohms -> 150; device rcl:R-US_0204/5 -> rcl:R-US_R0603
- R2: value 10K Ohms -> 10K; device rcl:R-US_0204/5 -> rcl:R-US_R0603
- R6: value 1.7K Ohms -> 10K; device rcl:R-US_0204/5 -> rcl:R-US_R0603
- R7: value 1K Ohms -> 10K; device rcl:R-US_0204/5 -> rcl:R-US_R0603
Connections:
- removed net REGPOW: C2.1, C3.1, C4.1, C5.1, J2.VCC, M1.VCC, R2.2, U1.AVCC, U1.VCC@4, U1.VCC@6, U2.OUT, U3.VCC
- removed net UNREGPOW: C1.1, FLYBACK_DIODE1.GPIN, FLYBACK_DIODE2.GPIN, FLYBACK_DIODE3.GPIN, FLYBACK_DIODE4.GPIN, J1.+, MOTOR.+, MOTOR1.+, MOTOR2.+, MOTOR3.+, R6.1, U2.IN
- new net 3V3: C2.1, C3.1, C4.1, C5.1, C9.2, J2.VCC, M1.VCC, R6.2, U$1.VOUT, U1.AVCC, U1.VCC@4, U1.VCC@6, U3.VCC
- new net G_LED: LED2.A, U1.PC2(ADC2)
- new net N$3: LED3.C, R4.1
- new net N$4: LED2.C, R3.1
- new net N$5: LED1.C, R1.1
- new net R_LED: LED1.A, U1.PC1(ADC1)
- new net VBATT: C1.1, FLYBACK_DIODE1.GPIN, FLYBACK_DIODE2.GPIN, FLYBACK_DIODE3.GPIN, FLYBACK_DIODE4.GPIN, J1.+, MOTOR.+, MOTOR1.+, MOTOR2.+, MOTOR3.+, R9.1, U$1.VIN, U$1.~SHDN
- new net Y_LED: LED3.A, U1.PC3(ADC3)
- net GND: now also C9.1, R1.2, R10.1, R11.1, R2.1, R3.2, R4.2, R8.2, U$1.VSS; no longer R1.1, R3.1, R4.1, R5.1, U2.GND, U2.GND1
- net PWM1: now also R2.2; no longer R1.2
- net PWM2: now also R7.2; no longer R3.2
- net PWM3: now also R10.2; no longer R4.2
- net PWM4: now also R11.2; no longer R5.2
- net RST: now also R6.1; no longer R2.1
- net VDIV: now also R8.1, R9.2; no longer R6.2, R7.2
Other:
- moved on the sheet: C1, C2, C6, FLYBACK_DIODE1, FLYBACK_DIODE2, FLYBACK_DIODE3, FLYBACK_DIODE4, J1, R1, R2, R3, R4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

Commit message: updates
Parts:
- added C10, C11, C12, C13, C8: 100uF, rcl:C-USC1206
Connections:
- net GND: now also C10.2, C11.2, C12.2, C13.2, C8.2
- net VBATT: now also C10.1, C11.1, C12.1, C13.1, C8.1
Other:
- moved on the sheet: J2
Changed lines of the file:
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@@
 <part name="GND17" library="supply1" deviceset="GND" device=""/>
 <part name="C9" library="rcl" deviceset="C-US" device="C0603" value="10uF"/>
+<part name="C8" library="rcl" deviceset="C-US" device="C1206" value="100uF"/>
+<part name="C10" library="rcl" deviceset="C-US" device="C1206" value="100uF"/>
+<part name="C11" library="rcl" deviceset="C-US" device="C1206" value="100uF"/>
+<part name="C12" library="rcl" deviceset="C-US" device="C1206" value="100uF"/>
+<part name="C13" library="rcl" deviceset="C-US" device="C1206" value="100uF"/>
 </parts>
 <sheets>
@@
 <instance part="U3" gate="G$1" x="33.02" y="104.14"/>
 <instance part="GND14" gate="1" x="5.08" y="73.66"/>
-<instance part="J2" gate="G$1" x="30.48" y="48.26"/>
-<instance part="GND15" gate="1" x="25.4" y="35.56"/>
+<instance part="J2" gate="G$1" x="66.04" y="55.88"/>
+<instance part="GND15" gate="1" x="60.96" y="43.18"/>
 <instance part="C6" gate="G$1" x="-88.9" y="119.38" rot="R90"/>
 <instance part="C7" gate="G$1" x="-109.22" y="91.44" rot="R270"/>
@@
 <instance part="GND17" gate="1" x="-20.32" y="127"/>
 <instance part="C9" gate="G$1" x="-220.98" y="73.66"/>
+<instance part="C8" gate="G$1" x="-248.92" y="132.08" rot="R270"/>
+<instance part="C10" gate="G$1" x="-162.56" y="-7.62"/>
+<instance part="C11" gate="G$1" x="-91.44" y="-10.16"/>
+<instance part="C12" gate="G$1" x="-20.32" y="-10.16"/>
+<instance part="C13" gate="G$1" x="50.8" y="-12.7"/>
 </instances>
 <busses>
@@
 <wire x1="-182.88" y1="22.86" x2="-200.66" y2="22.86" width="0.1524" layer="91"/>
 <wire x1="-200.66" y1="22.86" x2="-200.66" y2="15.24" width="0.1524" layer="91"/>
+<pinref part="C10" gate="G$1" pin="1"/>
+<wire x1="-162.56" y1="-5.08" x2="-162.56" y2="22.86" width="0.1524" layer="91"/>
+<wire x1="-162.56" y1="22.86" x2="-175.26" y2="22.86" width="0.1524" layer="91"/>
+<junction x="-175.26" y="22.86"/>
 </segment>
 <segment>
@@
 <wire x1="-109.22" y1="22.86" x2="-127" y2="22.86" width="0.1524" layer="91"/>
 <wire x1="-127" y1="22.86" x2="-127" y2="15.24" width="0.1524" layer="91"/>
+<pinref part="C11" gate="G$1" pin="1"/>
+<wire x1="-91.44" y1="-7.62" x2="-91.44" y2="22.86" width="0.1524" layer="91"/>
+<wire x1="-91.44" y1="22.86" x2="-101.6" y2="22.86" width="0.1524" layer="91"/>
+<junction x="-101.6" y="22.86"/>
 </segment>
 <segment>
@@
 <wire x1="-38.1" y1="22.86" x2="-55.88" y2="22.86" width="0.1524" layer="91"/>
 <wire x1="-55.88" y1="22.86" x2="-55.88" y2="15.24" width="0.1524" layer="91"/>
+<pinref part="C12" gate="G$1" pin="1"/>
+<wire x1="-20.32" y1="-7.62" x2="-20.32" y2="22.86" width="0.1524" layer="91"/>
+<wire x1="-20.32" y1="22.86" x2="-30.48" y2="22.86" width="0.1524" layer="91"/>
+<junction x="-30.48" y="22.86"/>
 </segment>
 <segment>
@@
 <wire x1="30.48" y1="20.32" x2="12.7" y2="20.32" width="0.1524" layer="91"/>
 <wire x1="12.7" y1="20.32" x2="12.7" y2="12.7" width="0.1524" layer="91"/>
+<pinref part="C13" gate="G$1" pin="1"/>
+<wire x1="50.8" y1="-10.16" x2="50.8" y2="20.32" width="0.1524" layer="91"/>
+<wire x1="50.8" y1="20.32" x2="38.1" y2="20.32" width="0.1524" layer="91"/>
+<junction x="38.1" y="20.32"/>
 </segment>
 <segment>
@@
 <pinref part="J1" gate="G$1" pin="+"/>
 <wire x1="-243.84" y1="144.78" x2="-243.84" y2="137.16" width="0.1524" layer="91"/>
-<wire x1="-243.84" y1="137.16" x2="-243.84" y2="124.46" width="0.1524" layer="91"/>
+<wire x1="-243.84" y1="137.16" x2="-243.84" y2="132.08" width="0.1524" layer="91"/>
 <label x="-243.84" y="144.78" size="1.778" layer="95" xref="yes"/>
+<wire x1="-243.84" y1="132.08" x2="-243.84" y2="124.46" width="0.1524" layer="91"/>
 <wire x1="-243.84" y1="124.46" x2="-243.84" y2="119.38" width="0.1524" layer="91"/>
 <wire x1="-243.84" y1="119.38" x2="-243.84" y2="116.84" width="0.1524" layer="91"/>
@@
 <junction x="-243.84" y="119.38"/>
 <pinref part="R9" gate="G$1" pin="1"/>
+<pinref part="C8" gate="G$1" pin="1"/>
+<wire x1="-246.38" y1="132.08" x2="-243.84" y2="132.08" width="0.1524" layer="91"/>
+<junction x="-243.84" y="132.08"/>
 </segment>
 </net>
@@
 <pinref part="J1" gate="G$1" pin="-"/>
 <wire x1="-254" y1="144.78" x2="-246.38" y2="144.78" width="0.1524" layer="91"/>
-<wire x1="-254" y1="144.78" x2="-254" y2="104.14" width="0.1524" layer="91"/>
+<wire x1="-254" y1="144.78" x2="-254" y2="132.08" width="0.1524" layer="91"/>
+<wire x1="-254" y1="132.08" x2="-254" y2="104.14" width="0.1524" layer="91"/>
 <wire x1="-254" y1="104.14" x2="-243.84" y2="104.14" width="0.1524" layer="91"/>
 <wire x1="-254" y1="144.78" x2="-254" y2="157.48" width="0.1524" layer="91"/>
@@
 <junction x="-243.84" y="104.14"/>
 <junction x="-238.76" y="104.14"/>
+<pinref part="C8" gate="G$1" pin="2"/>
+<junction x="-254" y="132.08"/>
 </segment>
 <segment>
@@
 <segment>
 <pinref part="MOSFET3" gate="G$1" pin="S"/>
-<wire x1="-55.88" y1="-20.32" x2="-55.88" y2="-40.64" width="0.1524" layer="91"/>
+<wire x1="-55.88" y1="-20.32" x2="-55.88" y2="-33.02" width="0.1524" layer="91"/>
 <pinref part="GND5" gate="1" pin="GND"/>
+<pinref part="C12" gate="G$1" pin="2"/>
+<wire x1="-55.88" y1="-33.02" x2="-55.88" y2="-40.64" width="0.1524" layer="91"/>
+<wire x1="-20.32" y1="-15.24" x2="-20.32" y2="-33.02" width="0.1524" layer="91"/>
+<wire x1="-20.32" y1="-33.02" x2="-55.88" y2="-33.02" width="0.1524" layer="91"/>
+<junction x="-55.88" y="-33.02"/>
 </segment>
 <segment>
@@
 <pinref part="GND1" gate="1" pin="GND"/>
 <pinref part="MOSFET1" gate="G$1" pin="S"/>
-<wire x1="-200.66" y1="-40.64" x2="-200.66" y2="-20.32" width="0.1524" layer="91"/>
+<wire x1="-200.66" y1="-40.64" x2="-200.66" y2="-35.56" width="0.1524" layer="91"/>
+<pinref part="C10" gate="G$1" pin="2"/>
+<wire x1="-200.66" y1="-35.56" x2="-200.66" y2="-20.32" width="0.1524" layer="91"/>
+<wire x1="-162.56" y1="-12.7" x2="-162.56" y2="-35.56" width="0.1524" layer="91"/>
+<wire x1="-162.56" y1="-35.56" x2="-200.66" y2="-35.56" width="0.1524" layer="91"/>
+<junction x="-200.66" y="-35.56"/>
 </segment>
 <segment>
@@
 <pinref part="GND3" gate="1" pin="GND"/>
 <pinref part="MOSFET2" gate="G$1" pin="S"/>
-<wire x1="-127" y1="-40.64" x2="-127" y2="-20.32" width="0.1524" layer="91"/>
+<wire x1="-127" y1="-40.64" x2="-127" y2="-30.48" width="0.1524" layer="91"/>
+<pinref part="C11" gate="G$1" pin="2"/>
+<wire x1="-127" y1="-30.48" x2="-127" y2="-20.32" width="0.1524" layer="91"/>
+<wire x1="-91.44" y1="-15.24" x2="-91.44" y2="-30.48" width="0.1524" layer="91"/>
+<wire x1="-91.44" y1="-30.48" x2="-127" y2="-30.48" width="0.1524" layer="91"/>
+<junction x="-127" y="-30.48"/>
 </segment>
 <segment>
@@
 <pinref part="GND7" gate="1" pin="GND"/>
 <pinref part="MOSFET4" gate="G$1" pin="S"/>
-<wire x1="12.7" y1="-43.18" x2="12.7" y2="-22.86" width="0.1524" layer="91"/>
+<wire x1="12.7" y1="-43.18" x2="12.7" y2="-35.56" width="0.1524" layer="91"/>
+<pinref part="C13" gate="G$1" pin="2"/>
+<wire x1="12.7" y1="-35.56" x2="12.7" y2="-22.86" width="0.1524" layer="91"/>
+<wire x1="50.8" y1="-17.78" x2="50.8" y2="-35.56" width="0.1524" layer="91"/>
+<wire x1="50.8" y1="-35.56" x2="12.7" y2="-35.56" width="0.1524" layer="91"/>
+<junction x="12.7" y="-35.56"/>
 </segment>
 <segment>
@@
 <pinref part="GND15" gate="1" pin="GND"/>
 <pinref part="J2" gate="G$1" pin="GND"/>
-<wire x1="25.4" y1="38.1" x2="25.4" y2="40.64" width="0.1524" layer="91"/>
+<wire x1="60.96" y1="45.72" x2="60.96" y2="48.26" width="0.1524" layer="91"/>
 <pinref part="J2" gate="G$1" pin="CTS"/>
-<wire x1="25.4" y1="40.64" x2="25.4" y2="43.18" width="0.1524" layer="91"/>
-<junction x="25.4" y="40.64"/>
+<wire x1="60.96" y1="48.26" x2="60.96" y2="50.8" width="0.1524" layer="91"/>
+<junction x="60.96" y="48.26"/>
 </segment>
 <segment>
@@
 <segment>
 <pinref part="J2" gate="G$1" pin="VCC"/>
-<wire x1="25.4" y1="45.72" x2="20.32" y2="45.72" width="0.1524" layer="91"/>
-<label x="20.32" y="45.72" size="1.778" layer="95" rot="R180" xref="yes"/>
+<wire x1="60.96" y1="53.34" x2="55.88" y2="53.34" width="0.1524" layer="91"/>
+<label x="55.88" y="53.34" size="1.778" layer="95" rot="R180" xref="yes"/>
 </segment>
 </net>
@@
 <segment>
 <pinref part="J2" gate="G$1" pin="TXO"/>
-<wire x1="25.4" y1="50.8" x2="20.32" y2="50.8" width="0.1524" layer="91"/>
-<label x="20.32" y="50.8" size="1.778" layer="95" rot="R180" xref="yes"/>
+<wire x1="60.96" y1="58.42" x2="55.88" y2="58.42" width="0.1524" layer="91"/>
+<label x="55.88" y="58.42" size="1.778" layer="95" rot="R180" xref="yes"/>
 </segment>
 </net>
@@
 <segment>
 <pinref part="J2" gate="G$1" pin="RXI"/>
-<wire x1="25.4" y1="48.26" x2="5.08" y2="48.26" width="0.1524" layer="91"/>
-<label x="5.08" y="48.26" size="1.778" layer="95" rot="R180" xref="yes"/>
+<wire x1="60.96" y1="55.88" x2="40.64" y2="55.88" width="0.1524" layer="91"/>
+<label x="40.64" y="55.88" size="1.778" layer="95" rot="R180" xref="yes"/>
 </segment>
 </net>
@@
 <segment>
 <pinref part="J2" gate="G$1" pin="DTR"/>
-<wire x1="25.4" y1="53.34" x2="2.54" y2="53.34" width="0.1524" layer="91"/>
-<label x="2.54" y="53.34" size="1.778" layer="95" rot="R180" xref="yes"/>
-</segment>
-</net>
+<wire x1="60.96" y1="60.96" x2="38.1" y2="60.96" width="0.1524" layer="91"/>
+<label x="38.1" y="60.96" size="1.778" layer="95" rot="R180" xref="yes"/>
+</segment>
+</net>
