File: QuadcopterHardware/Quadcopter/Quadcopter.brd (EAGLE design)
At the start: 47 x 28 mm, 47 parts, among them J2 FTDI_DEVICERA_SMT, M1 WIRELESS-NRF24L01, U1 ATMEGA328P_TQFP, U3 GY-521MPU6050

Commit message: almost there
Parts:
- moved C14 67.5 mm to (5.56, 23.7), turned to 90 degrees
- moved C9 63.7 mm to (3.25, 23.7), turned to 90 degrees
- moved R8 35.9 mm to (34.4, 22.5), turned to 90 degrees
- moved R9 29.4 mm to (33.9, 19.2), turned to 90 degrees
- moved R6 26.6 mm to (8.43, 11.6), turned to 0 degrees
- moved C6 11.3 mm to (8.41, 13.9), turned to 0 degrees
Routing:
- net 3V3: track 64.9 -> 77.6 mm
- net DTR: track 0.00 -> 11.6 mm, vias 0 -> 1
- net GND: track 36.3 -> 46.9 mm, vias 3 -> 4
- net RST: track 0.05 -> 9.72 mm
- net VDIV: track 0.00 -> 7.76 mm
- net VBATT: track 67.1 -> 73.2 mm
Changed lines of the file:
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@@
 <element name="C12" library="rcl" package="C1210" value="100uF" x="28.03" y="8.05"/>
 <element name="C13" library="rcl" package="C1210" value="100uF" x="37.16" y="9.55"/>
-<element name="C14" library="rcl" package="C0603" value="100nF" x="70.22" y="43.25"/>
+<element name="C14" library="rcl" package="C0603" value="100nF" x="5.5625" y="23.72" rot="R90"/>
 <element name="C2" library="rcl" package="C0603" value="1uF" x="39.48" y="15.5"/>
 <element name="C3" library="rcl" package="C0603" value="100nF" x="16.54" y="17.35" rot="R180"/>
 <element name="C4" library="rcl" package="C0603" value="100nF" x="31.84" y="14.15"/>
 <element name="C5" library="rcl" package="C0603" value="100nF" x="16.53" y="15.1" rot="R180"/>
-<element name="C6" library="rcl" package="C0603" value="100nF" x="16.15" y="22.1" rot="R180"/>
+<element name="C6" library="rcl" package="C0603" value="100nF" x="8.4125" y="13.9"/>
 <element name="C7" library="rcl" package="C0603" value="100nF" x="31.73" y="16.4"/>
 <element name="C8" library="rcl" package="C1210" value="100uF" x="38.7" y="22.89" rot="R90"/>
-<element name="C9" library="rcl" package="C0603" value="10uF" x="63.87" y="43.25"/>
+<element name="C9" library="rcl" package="C0603" value="10uF" x="3.25" y="23.745" rot="R90"/>
 <element name="FLYBACK_DIODE1" library="quad" package="MINI2-F3-B" value="DB2W40300L" x="8.23" y="3.08" rot="MR0"/>
 <element name="FLYBACK_DIODE2" library="quad" package="MINI2-F3-B" value="DB2W40300L" x="17.31" y="3.08" rot="MR0"/>
@@
 <element name="R3" library="rcl" package="R0603" value="150" x="88.91" y="22.58"/>
 <element name="R4" library="rcl" package="R0603" value="150" x="88.83" y="18.08"/>
-<element name="R6" library="rcl" package="R0603" value="10K" x="32.95" y="22" rot="R180"/>
+<element name="R6" library="rcl" package="R0603" value="10K" x="8.425" y="11.625"/>
 <element name="R7" library="rcl" package="R0603" value="10K" x="24" y="6.53" rot="R270"/>
-<element name="R8" library="rcl" package="R0603" value="1K" x="36.77" y="58.33"/>
-<element name="R9" library="rcl" package="R0603" value="1.7K" x="41.79" y="47.5"/>
+<element name="R8" library="rcl" package="R0603" value="1K" x="34.42" y="22.4575" rot="R90"/>
+<element name="R9" library="rcl" package="R0603" value="1.7K" x="33.9375" y="19.165" rot="R90"/>
 <element name="RES1" library="quad" package="CSTCE16M0V53-R0" value="CSTCE10M0G55-R0" x="18.97" y="12.38" rot="R270"/>
 <element name="S1" library="quad" package="TACTILE-SWITCH-SMD" value="SWITCH-MOMENTARY-2SMD" x="3.9" y="7.15" rot="R270">
@@
 <wire x1="35.76" y1="9.55" x2="35.76" y2="7.86" width="1.016" layer="1"/>
 <wire x1="35.76" y1="7.86" x2="37.73" y2="5.89" width="1.016" layer="1"/>
-<wire x1="43.25" y1="23.79" x2="40.94" y2="47.5" width="0" layer="19" extent="1-1"/>
+<wire x1="33.9375" y1="18.315" x2="34.1275" y2="18.315" width="0.4064" layer="1"/>
+<wire x1="34.1275" y1="18.315" x2="36.8125" y2="21" width="0.4064" layer="1"/>
+<wire x1="36.8125" y1="21" x2="38.21" y2="21" width="0.4064" layer="1"/>
+<wire x1="38.21" y1="21" x2="38.7" y2="21.49" width="0.4064" layer="1"/>
 </signal>
 <signal name="GND">
@@
 <wire x1="15.69" y1="17.35" x2="15.69" y2="17.69" width="0.4064" layer="1"/>
 <wire x1="15.69" y1="17.69" x2="17" y2="19" width="0.4064" layer="1"/>
+<wire x1="34.42" y1="23.3075" x2="36.63" y2="23.3075" width="0.4064" layer="1"/>
+<wire x1="36.63" y1="23.3075" x2="36.75" y2="23.1875" width="0.4064" layer="1"/>
+<via x="5.625" y="7.625" extent="1-16" drill="0.6"/>
+<wire x1="5.805" y1="9.944" x2="5.805" y2="7.805" width="0.4064" layer="1"/>
+<wire x1="5.805" y1="7.805" x2="5.625" y2="7.625" width="0.4064" layer="1"/>
+<wire x1="5.5625" y1="24.57" x2="5.57" y2="24.57" width="0.4064" layer="1"/>
+<wire x1="5.57" y1="24.57" x2="6.5625" y2="25.5625" width="0.4064" layer="1"/>
+<wire x1="6.5625" y1="25.5625" x2="8.4525" y2="25.5625" width="0.4064" layer="1"/>
+<wire x1="8.4525" y1="25.5625" x2="8.63" y2="25.74" width="0.4064" layer="1"/>
+<wire x1="3.25" y1="24.595" x2="5.5375" y2="24.595" width="0.4064" layer="1"/>
+<wire x1="5.5375" y1="24.595" x2="5.5625" y2="24.57" width="0.4064" layer="1"/>
 <wire x1="89.76" y1="22.58" x2="89.84" y2="26.08" width="0" layer="19" extent="1-1"/>
 <wire x1="89.68" y1="18.08" x2="89.76" y2="22.58" width="0" layer="19" extent="1-1"/>
-<wire x1="71.07" y1="43.25" x2="89.84" y2="26.08" width="0" layer="19" extent="1-1"/>
-<wire x1="64.72" y1="43.25" x2="71.07" y2="43.25" width="0" layer="19" extent="1-1"/>
-<wire x1="43.25" y1="22.09" x2="64.72" y2="43.25" width="0" layer="19" extent="1-1"/>
-<wire x1="5.805" y1="9.944" x2="11.17" y2="8.3" width="0" layer="19" extent="1-1"/>
-<wire x1="37.62" y1="58.33" x2="64.72" y2="43.25" width="0" layer="19" extent="1-1"/>
+<wire x1="43.25" y1="22.09" x2="89.76" y2="22.58" width="0" layer="19" extent="1-1"/>
+<wire x1="40.2916" y1="18.25" x2="42.99" y2="19.7" width="0" layer="19" extent="1-1"/>
 </signal>
 <signal name="3V3">
@@
 <wire x1="36" y1="18.25" x2="23" y2="18.25" width="0.4064" layer="16"/>
 <wire x1="23" y1="18.25" x2="21.875" y2="17.125" width="0.4064" layer="16"/>
-<wire x1="63.02" y1="43.25" x2="69.37" y2="43.25" width="0" layer="19" extent="1-1"/>
-<wire x1="36.6086" y1="18.25" x2="63.02" y2="43.25" width="0" layer="19" extent="1-1"/>
-<wire x1="32.1" y1="22" x2="36" y2="18.25" width="0" layer="19" extent="1-16"/>
-<wire x1="14.5" y1="25.1" x2="17.39" y2="17.35" width="0" layer="19" extent="1-1"/>
-<wire x1="11.17" y1="25.74" x2="14.5" y2="25.1" width="0" layer="19" extent="1-1"/>
-<wire x1="2.98" y1="18.39" x2="11.17" y2="25.74" width="0" layer="19" extent="16-16"/>
+<wire x1="5.5625" y1="22.87" x2="6.12" y2="22.87" width="0.4064" layer="1"/>
+<wire x1="6.12" y1="22.87" x2="7.75" y2="24.5" width="0.4064" layer="1"/>
+<wire x1="7.75" y1="24.5" x2="9.93" y2="24.5" width="0.4064" layer="1"/>
+<wire x1="9.93" y1="24.5" x2="11.17" y2="25.74" width="0.4064" layer="1"/>
+<wire x1="11.17" y1="25.74" x2="11.9475" y2="25.74" width="0.4064" layer="1"/>
+<wire x1="11.9475" y1="25.74" x2="12.625" y2="25.0625" width="0.4064" layer="1"/>
+<wire x1="12.625" y1="25.0625" x2="14.4625" y2="25.0625" width="0.4064" layer="1"/>
+<wire x1="14.4625" y1="25.0625" x2="14.5" y2="25.1" width="0.4064" layer="1"/>
+<wire x1="14.4625" y1="25.0625" x2="17.39" y2="17.35" width="0" layer="19" extent="1-1"/>
+<wire x1="2.98" y1="18.39" x2="3.25" y2="22.895" width="0" layer="19" extent="1-16"/>
+<wire x1="9.275" y1="11.625" x2="17.38" y2="15.1" width="0" layer="19" extent="1-1"/>
+<wire x1="3.25" y1="22.895" x2="5.5375" y2="22.895" width="0.4064" layer="1"/>
+<wire x1="5.5375" y1="22.895" x2="5.5625" y2="22.87" width="0.4064" layer="1"/>
 </signal>
 <signal name="RST">
@@
 <contactref element="R6" pad="1"/>
 <wire x1="1.995" y1="9.944" x2="1.95" y2="9.944" width="0.4064" layer="1"/>
-<wire x1="23.9" y1="20.8526" x2="33.8" y2="22" width="0" layer="19" extent="1-1"/>
-<wire x1="17" y1="22.1" x2="23.9" y2="20.8526" width="0" layer="19" extent="1-1"/>
-<wire x1="1.995" y1="9.944" x2="17" y2="22.1" width="0" layer="19" extent="1-1"/>
+<wire x1="7.575" y1="11.625" x2="7.575" y2="13.375" width="0.4064" layer="1"/>
+<wire x1="7.575" y1="13.375" x2="7.575" y2="13.8875" width="0.4064" layer="1"/>
+<wire x1="7.575" y1="13.8875" x2="7.5625" y2="13.9" width="0.4064" layer="1"/>
+<wire x1="1.995" y1="9.944" x2="1.995" y2="10.62" width="0.4064" layer="1"/>
+<wire x1="1.995" y1="10.62" x2="3.25" y2="11.875" width="0.4064" layer="1"/>
+<wire x1="3.25" y1="11.875" x2="6.075" y2="11.875" width="0.4064" layer="1"/>
+<wire x1="6.075" y1="11.875" x2="7.575" y2="13.375" width="0.4064" layer="1"/>
+<wire x1="7.5625" y1="13.9" x2="23.9" y2="20.8526" width="0" layer="19" extent="1-1"/>
 </signal>
 <signal name="MISO">
@@
 <contactref element="C6" pad="2"/>
 <contactref element="J2" pad="1"/>
-<wire x1="2.98" y1="10.77" x2="15.3" y2="22.1" width="0" layer="19" extent="1-16"/>
+<wire x1="9.2625" y1="13.9" x2="9.9125" y2="13.9" width="0.4064" layer="1"/>
+<wire x1="9.9125" y1="13.9" x2="11.25" y2="12.5625" width="0.4064" layer="1"/>
+<via x="11.25" y="12.5625" extent="1-16" drill="0.6"/>
+<wire x1="2.98" y1="10.77" x2="9.4575" y2="10.77" width="0.4064" layer="16"/>
+<wire x1="9.4575" y1="10.77" x2="11.25" y2="12.5625" width="0.4064" layer="16"/>
 </signal>
 <signal name="CSN">
@@
 <contactref element="R8" pad="1"/>
 <contactref element="R9" pad="2"/>
-<wire x1="42.64" y1="47.5" x2="35.92" y2="58.33" width="0" layer="19" extent="1-1"/>
-<wire x1="28.5926" y1="18.56" x2="42.64" y2="47.5" width="0" layer="19" extent="1-1"/>
+<wire x1="34.42" y1="21.6075" x2="34.4375" y2="21.6075" width="0.4064" layer="1"/>
+<wire x1="34.4375" y1="21.6075" x2="34.4375" y2="20.515" width="0.4064" layer="1"/>
+<wire x1="34.4375" y1="20.515" x2="33.9375" y2="20.015" width="0.4064" layer="1"/>
+<wire x1="28.5926" y1="18.56" x2="32.4825" y2="18.56" width="0.4064" layer="1"/>
+<wire x1="32.4825" y1="18.56" x2="33.9375" y2="20.015" width="0.4064" layer="1"/>
 </signal>
 <signal name="N$3">
