File: QuadcopterHardware/Quadcopter/v3/Quadcopter_v3.brd (EAGLE design)
At the start: 47 x 28 mm, 43 parts, among them J1 FTDI_DEVICE, M1 WIRELESS-NRF24L01, U1 ATMEGA328P_TQFP, U3 GY-521MPU6050

Commit message: final (cullen rev)
Parts:
- moved R6 34.0 mm to (11.0, 24.9), flipped to the bottom, turned to 0 degrees
- moved C6 33.2 mm to (14.1, 24.9), flipped to the bottom, turned to 180 degrees
Routing:
- net 3V3: track 130.1 -> 65.4 mm, vias 1 -> 0
- net DTR: track 47.6 -> 2.25 mm, vias 1 -> 0
- net CSN: track 26.9 -> 37.0 mm, vias 1 -> 2
- net RST: track 41.6 -> 47.6 mm, vias 1 -> 2
- net VBATT: track 74.9 -> 76.0 mm, vias 4 -> 2
- net CE: track 40.0 -> 39.1 mm
- net SCK: track 19.0 -> 18.3 mm
- net UART_RX: track 16.6 -> 16.0 mm
- added copper zone on layer 1, net 3V3
